File: ilse.kicad_sch (KiCad schematic)
At the start: 91 parts, among them J1 OUT, J2 EURO RACK POWER, J3 CV Inputs, J4 1V/Oct, J5 Gate, J6 Cutoff, J7 Filter In, Q1 BC560, Q2 BC560, Q3 BC560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

Commit message: include manf# for rev2
Parts:
- BT1, BT2: value 9 V -> 100; manf# (none) -> 36-232-ND
- C1, C11, C5: manf# (none) -> FG28X5R1H105KRT06
- C10: manf# (none) -> SR215C102KAR
- C12, C13: manf# (none) -> ECE-A1HKS100
- C2, C6: manf# (none) -> C322C104K5R5TA7305
- C3, C4: manf# (none) -> C317C103K5R5TA
- C7, C8, C9: manf# (none) -> C322C473K5R5TA7301
- D1, D2: manf# (none) -> WP710A10LID, L424SRDT
- D3, D4, D5: manf# (none) -> 1N5819_R2_00001
- J1, J4, J5, J6, J7: manf# (none) -> PJ398SM
- J2: manf# (none) -> 302-S101
- J3: manf# (none) -> PH2-06-UA
- JP1: manf# (none) -> STC02SYAN
- Q1, Q2, Q3: value BC560 -> BC559; manf# (none) -> BC559BTA
- Q4, Q5, Q6: value BC550 -> BC548; manf# (none) -> BC548BTA
- R1, R12, R34: manf# (none) -> CF18JT4K70
- R10, R11, R2, R21, R22, R23, R29, R37: manf# (none) -> RNF14FTD47K0
- R13, R14, R17, R18, R20, R24, R25, R27, R28, R3, R36, R38, R39, R4, R8: manf# (none) -> RR03J100KTB
- R15: manf# (none) -> CF18JT1K50
- R16, R35, R5, R6, R9: manf# (none) -> RNF14FTD1K00
- R19, R26, R30, R32, R33, R40: manf# (none) -> RNF14FTD10K0
- R31: manf# (none) -> CF18JT2K20
- R7: value 20k -> 22k; manf# (none) -> CF14JT22K0
- RV3: manf# (none) -> 67YR500LF
- U1, U2: manf# (none) -> TL074CN
