File: ilse.kicad_pcb (KiCad board)
At the start: 2 copper layers, 80.9 x 109.5 mm, 87 parts, among them J1 OUT, J2 EURO RACK POWER, J3 CV Inputs, J4 1V/Oct, J5 Gate, J6 Cutoff, J7 Filter In, Q1 BC559, Q2 BC559, Q3 BC559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

Commit message: started frontpanel file
Parts:
- moved RV3 7.66 mm to (167.7, 121.4), turned to 0 degrees
Routing:
- net Net-(R15-Pad2): track 18.3 -> 11.7 mm
Other:
- board size 80.9 x 109.5 mm -> 78.5 x 109.5 mm

Commit message: holes completed on frontpanel
Parts:
- J3: moved to B.Cu
- moved D1 32.9 mm to (131.0, 42.8)
- moved R12 32.6 mm to (136.7, 52.3)
- moved LOGO1 30.4 mm to (161.7, 46.8)
- moved J3 2.30 mm to (146.1, 62.5), turned to 0 degrees
Routing:
- net VCC: track 266.0 -> 237.3 mm
- net Osc 2 Detune: track 48.2 -> 55.7 mm
- net VSS: track 203.3 -> 197.1 mm, vias 3 -> 4
- net GATE: track 68.3 -> 64.7 mm, vias 1 -> 0
- net 1V/Oct: track 142.4 -> 139.1 mm
- net Freq CV: track 136.6 -> 134.1 mm
- net Filter Cutoff: track 76.4 -> 78.7 mm
- net LFO Speed: track 33.7 -> 35.8 mm
- net GND: vias 95 -> 139
Other:
- board text removed: "Ilse"
